Commit message: refactor():添加了机械臂的moveit和urdf

File: src/robot_description/nero_description/urdf/nero_description.urdf (robot description, URDF)
Before this commit: robot nero_description, 10 links, 9 joints
Links:
- removed link end_effector
- added link link8
Joints:
- removed joint end_effector_joint
- added joint joint8: type fixed, parent link7, child link8, origin xyz=0.00000000 0.00000000 -0.02350000 rpy=0 0 0
